File: BOARD DESIGN/iTilt8.brd (EAGLE design)
At the start: 0 parts

Commit message: Add files via upload
Routing:
- net S$61: track 19.2 -> 0.00 mm
- net S$53: track 18.5 -> 0.00 mm
- net S$83: track 0.00 -> 4.45 mm
- net S$63: track 4.45 -> 0.00 mm
- net S$33: track 22.2 -> 25.3 mm
- net S$39: track 12.3 -> 15.0 mm
- net S$50: track 2.54 -> 0.00 mm
- net S$43: track 2.54 -> 0.00 mm
Changed lines of the file:
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@@
 <hole x="6.35" y="29.21" drill="0.6"/>
 <hole x="6.35" y="67.31" drill="0.6"/>
-<hole x="8.89" y="7.62" drill="1"/>
-<hole x="13.97" y="7.62" drill="1"/>
+<hole x="15.24" y="7.62" drill="1"/>
+<hole x="20.32" y="7.62" drill="1"/>
 <hole x="25.4" y="30.48" drill="0.6"/>
 <hole x="25.4" y="34.29" drill="0.6"/>
-<hole x="8.89" y="15.24" drill="1"/>
-<hole x="13.97" y="15.24" drill="1"/>
+<hole x="15.24" y="15.24" drill="1"/>
+<hole x="20.32" y="15.24" drill="1"/>
 <hole x="22.225" y="34.29" drill="0.6"/>
 <hole x="29.21" y="92.71" drill="0.6"/>
@@
 <hole x="5.08" y="121.92" drill="0.6"/>
 <hole x="15.24" y="34.29" drill="0.6"/>
-<hole x="15.24" y="26.67" drill="0.6"/>
-<hole x="20.955" y="8.255" drill="0.6"/>
-<hole x="26.67" y="8.255" drill="0.6"/>
 <hole x="23.495" y="41.91" drill="0.6"/>
 <hole x="25.4" y="38.1" drill="0.6"/>
@@
 </signal>
 <signal name="S$68">
-<wire x1="13.97" y1="6.35" x2="13.97" y2="8.255" width="2.54" layer="16"/>
+<wire x1="20.32" y1="6.35" x2="20.32" y2="8.255" width="2.54" layer="16"/>
 </signal>
 <signal name="S$14">
-<wire x1="13.97" y1="16.51" x2="13.97" y2="14.605" width="2.54" layer="16"/>
+<wire x1="20.32" y1="16.51" x2="20.32" y2="14.605" width="2.54" layer="16"/>
 </signal>
 <signal name="S$51">
@@
 </signal>
 <signal name="S$40">
-<wire x1="8.89" y1="8.255" x2="8.89" y2="6.35" width="2.54" layer="16"/>
+<wire x1="15.24" y1="8.255" x2="15.24" y2="6.35" width="2.54" layer="16"/>
 </signal>
 <signal name="S$45">
-<wire x1="8.89" y1="16.51" x2="8.89" y2="14.605" width="2.54" layer="16"/>
+<wire x1="15.24" y1="16.51" x2="15.24" y2="14.605" width="2.54" layer="16"/>
 </signal>
 <signal name="S$36">
 <wire x1="26.035" y1="30.48" x2="21.59" y2="30.48" width="2.54" layer="16"/>
 </signal>
-<signal name="S$63">
+<signal name="S$83">
 <wire x1="21.59" y1="34.29" x2="26.035" y2="34.29" width="2.54" layer="16"/>
 </signal>
@@
 <wire x1="9.525" y1="36.83" x2="7.62" y2="36.83" width="0.8128" layer="16"/>
 <wire x1="9.525" y1="29.21" x2="9.525" y2="36.83" width="0.8128" layer="16"/>
-<wire x1="13.335" y1="17.145" x2="9.525" y2="29.21" width="0.8128" layer="16"/>
+<wire x1="19.685" y1="17.145" x2="9.525" y2="29.21" width="0.8128" layer="16"/>
 </signal>
 <signal name="S$39">
-<wire x1="6.35" y1="28.575" x2="8.89" y2="16.51" width="0.8128" layer="16"/>
+<wire x1="6.35" y1="28.575" x2="15.24" y2="16.51" width="0.8128" layer="16"/>
 </signal>
 <signal name="S$69">
-<wire x1="8.89" y1="13.97" x2="8.89" y2="9.525" width="0.8128" layer="16"/>
+<wire x1="15.24" y1="13.97" x2="15.24" y2="9.525" width="0.8128" layer="16"/>
 </signal>
 <signal name="S$70">
-<wire x1="13.97" y1="13.335" x2="13.97" y2="9.525" width="0.8128" layer="16"/>
+<wire x1="20.32" y1="13.335" x2="20.32" y2="9.525" width="0.8128" layer="16"/>
 </signal>
 <signal name="S$42">
 <wire x1="28.575" y1="72.39" x2="29.845" y2="72.39" width="1.9304" layer="16"/>
-</signal>
-<signal name="S$50">
-<wire x1="26.67" y1="6.985" x2="26.67" y2="9.525" width="2.54" layer="16"/>
 </signal>
 <signal name="S$38">
@@
 <signal name="S$41">
 <wire x1="6.35" y1="104.775" x2="5.08" y2="104.775" width="1.6764" layer="16"/>
-</signal>
-<signal name="S$43">
-<wire x1="20.955" y1="9.525" x2="20.955" y2="6.985" width="2.54" layer="16"/>
-</signal>
-<signal name="S$53">
-<wire x1="15.875" y1="26.67" x2="14.605" y2="26.67" width="1.778" layer="16"/>
-<wire x1="20.955" y1="10.16" x2="15.875" y2="26.67" width="0.8128" layer="16"/>
 </signal>
 <signal name="S$54">
@@
 <wire x1="26.035" y1="45.72" x2="28.575" y2="44.45" width="0.8128" layer="16"/>
 </signal>
-<signal name="S$61">
-<wire x1="24.13" y1="29.21" x2="26.67" y2="10.16" width="0.8128" layer="16"/>
-</signal>
 <signal name="S$65">
